Commit message: [add]realsense model in gazebo

File: yumi_description/urdf/camera_base/camera_base.urdf.xacro (robot description, xacro)
@@ -31,5 +31,5 @@
 		</link>
 		<joint name="camera_base_link_joint_2" type="fixed">
-			<origin xyz="0.075 0.0 0" rpy="0.0 0 0.0"/>
+			<origin xyz="0.075 0.0 0" rpy="0.0 ${angle} 0.0"/>
 			<parent link="camera_base_link"/>
 			<child link="camera_base_2_link"/>
@@ -40,5 +40,5 @@
 					<mesh filename="package://yumi_description/meshes/camera_base/yumi_camera_base_2.STL"/>
 				</geometry>
-				<origin rpy="0 ${angle} 0" xyz="0 0 0" />
+				<origin rpy="0 0 0" xyz="0 0 0" />
 			</visual>
 			<collision>
@@ -46,8 +46,8 @@
 					<box size="0.25 0.015 0.015"/>
 				</geometry>
-				<origin xyz="0.125 0 0" rpy="0 ${angle} 0"/>
+				<origin xyz="0.125 0 0" rpy="0 0 0"/>
 			</collision>
 			<inertial>
-				<origin xyz="0.0 0.0 0.0" rpy="0.0 ${angle} 0.0"/>
+				<origin xyz="0.0 0.0 0.0" rpy="0.0 0.0 0.0"/>
 				<xacro:box_inertial mass="0.25" height="0.25" width="0.015" depth="0.015"/>
 			</inertial>

File: yumi_description/urdf/yumi.urdf (robot description, URDF)
Before this commit: robot yumi, 22 links, 21 joints
Links:
- added link base_footprint
- added link camera_base_2_link, mass 0.25; collision box size=0.25 0.015 0.015; visual mesh filename=package://yumi_description/meshes/camera_base/yumi_camera_b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
- added link camera_base_link, mass 0.2; collision box size=0.15 0.015 0.015; visual mesh filename=package://yumi_description/meshes/camera_base/yumi_camera_b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
- added link camera_bottom_screw_frame
- added link camera_color_frame
- added link camera_color_optical_frame
- added link camera_depth_frame
- added link camera_depth_optical_frame
- added link camera_infra1_frame
- added link camera_infra1_optical_frame
- added link camera_infra2_frame
- added link camera_infra2_optical_frame
- added link camera_link, mass 0.564; collision box size=0.02505 0.09 0.025; visual mesh filename=package://realsense2_description/meshes/d435.dae
- added link connect_base_link, mass 0.434; collision box size=0.17 0.17 0.015; visual mesh filename=package://lift_robot_description/meshes/stl/connect_base_v2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
- added link front_left_steering_link, mass 0.05; collision box size=0.07 0.07 0.07; visual mesh filename=package://lift_robot_description/meshes/stl/steering.STL
- added link front_left_wheel_link, mass 1.0; collision cylinder length=0.035 radius=0.035; visual mesh filename=package://lift_robot_description/meshes/stl/wheel_v2.STL
- added link front_right_steering_link, mass 0.05; collision box size=0.07 0.07 0.07; visual mesh filename=package://lift_robot_description/meshes/stl/steering.STL
- added link front_right_wheel_link, mass 1.0; collision cylinder length=0.035 radius=0.035; visual mesh filename=package://lift_robot_description/meshes/stl/wheel_v2.STL
- added link prop_link, mass 2.813; collision box size=0.075 0.075 0.5; visual mesh filename=package://lift_robot_description/meshes/stl/prop_v2.STL
- added link rear_left_steering_link, mass 0.05; collision box size=0.07 0.07 0.07; visual mesh filename=package://lift_robot_description/meshes/stl/steering.STL
- added link rear_left_wheel_link, mass 1.0; collision cylinder length=0.035 radius=0.035; visual mesh filename=package://lift_robot_description/meshes/stl/wheel_v2.STL
- added link rear_right_steering_link, mass 0.05; collision box size=0.07 0.07 0.07; visual mesh filename=package://lift_robot_description/meshes/stl/steering.STL
- added link rear_right_wheel_link, mass 1.0; collision cylinder length=0.035 radius=0.035; visual mesh filename=package://lift_robot_description/meshes/stl/wheel_v2.STL
- added link under_base_link, mass 40; collision box size=0.6 0.7 0.1; visual mesh filename=package://lift_robot_description/meshes/stl/under_base_v2.S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
- link gripper_l_finger_l: mass 0.01 -> 0.04
- link gripper_l_finger_r: mass 0.01 -> 0.04
- link gripper_r_finger_l: mass 0.01 -> 0.04
- link gripper_r_finger_r: mass 0.01 -> 0.04
Joints:
- added joint base_link_to_world_joint: type fixed, parent connect_base_link, child yumi_base_link, origin xyz=0 0 0.015
- added joint camera_base_link_joint: type fixed, parent yumi_base_link, child camera_base_link, origin xyz=-0.025 0.0 0.475  rpy=0  0 0
- added joint camera_base_link_joint_2: type fixed, parent camera_base_link, child camera_base_2_link, origin xyz=0.075 0.0 0 rpy=0.0 -0.785398163397 0.0
- added joint camera_color_joint: type fixed, parent camera_link, child camera_color_frame, origin xyz=0 0.015 0 rpy=0 0 0
- added joint camera_color_optical_joint: type fixed, parent camera_color_frame, child camera_color_optical_frame, origin xyz=0 0 0 rpy=-1.57079632679 0 -1.57079632679
- added joint camera_depth_joint: type fixed, parent camera_link, child camera_depth_frame, origin xyz=0 0 0 rpy=0 0 0
- added joint camera_depth_optical_joint: type fixed, parent camera_depth_frame, child camera_depth_optical_frame, origin xyz=0 0 0 rpy=-1.57079632679 0 -1.57079632679
- added joint camera_infra1_joint: type fixed, parent camera_link, child camera_infra1_frame, origin xyz=0 0.0 0 rpy=0 0 0
- added joint camera_infra1_optical_joint: type fixed, parent camera_infra1_frame, child camera_infra1_optical_frame, origin xyz=0 0 0 rpy=-1.57079632679 0 -1.57079632679
- added joint camera_infra2_joint: type fixed, parent camera_link, child camera_infra2_frame, origin xyz=0 -0.05 0 rpy=0 0 0
- added joint camera_infra2_optical_joint: type fixed, parent camera_infra2_frame, child camera_infra2_optical_frame, origin xyz=0 0 0 rpy=-1.57079632679 0 -1.57079632679
- added joint camera_joint: type fixed, parent camera_base_2_link, child camera_bottom_screw_frame, origin xyz=0.1 0 -0.02 rpy=0 1.57079632679 0
- added joint camera_link_joint: type fixed, parent camera_bottom_screw_frame, child camera_link, origin xyz=0.0106 0.0175 0.0125 rpy=0 0 0
- added joint connect_base_link_joint: type prismatic, parent prop_link, child connect_base_link, origin xyz=0.1455 0 0.025 rpy=0 0 0, axis 0 0 1, limit lower=0 upper=0.465 effort=1000.0 velocity=0.5
- added joint front_left_steering_joint: type revolute, parent under_base_link, child front_left_steering_link, origin xyz=0.3 0.25  0.07, axis 0 0 1, limit lower=-3.14159274 upper=3.14159274 effort=1000 velocity=1000
- added joint front_left_wheel_joint: type continuous, parent front_left_steering_link, child front_left_wheel_link, origin xyz=0 -0.0175 -0.045, axis 0 1 0, limit effort=0.4 velocity=12.0
- added joint front_right_steering_joint: type revolute, parent under_base_link, child front_right_steering_link, origin xyz=0.3 -0.25   0.07 rpy=0 0 0, axis 0 0 1, limit lower=-3.14159274 upper=3.14159274 effort=1000 velocity=1000
- added joint front_right_wheel_joint: type continuous, parent front_right_steering_link, child front_right_wheel_link, origin xyz=0 -0.0175 -0.045, axis 0 1 0, limit effort=0.4 velocity=12.0
- added joint prop_to_base_link_jiont: type fixed, parent under_base_link, child prop_link, origin xyz=0.1375 0 0.1 rpy=0 0 0
- added joint rear_left_steering_joint: type revolute, parent under_base_link, child rear_left_steering_link, origin xyz=-0.3 0.25  0.07, axis 0 0 1, limit lower=-3.14159274 upper=3.14159274 effort=1000 velocity=1000
- added joint rear_left_wheel_joint: type continuous, parent rear_left_steering_link, child rear_left_wheel_link, origin xyz=0 -0.0175 -0.045, axis 0 1 0, limit effort=0.4 velocity=12.0
- added joint rear_right_steering_joint: type revolute, parent under_base_link, child rear_right_steering_link, origin xyz=-0.3 -0.25  0.07 rpy=0 0 0, axis 0 0 1, limit lower=-3.14159274 upper=3.14159274 effort=1000 velocity=1000
- added joint rear_right_wheel_joint: type continuous, parent rear_right_steering_link, child rear_right_wheel_link, origin xyz=0 -0.0175 -0.045, axis 0 1 0, limit effort=0.4 velocity=12.0
- added joint under_base_link_joint: type fixed, parent base_footprint, child under_base_link, origin xyz=0 0 0.02

File: yumi_description/urdf/yumi.urdf.xacro (robot description, xacro)
@@ -11,6 +11,7 @@
   <!-- Import Gazebo plugins -->
   <xacro:include filename="$(find yumi_description)/urdf/Gazebo/gazebo.urdf.xacro"/>
-    <xacro:include filename="$(find  lift_robot_description)/robots/lift_robot.urdf_origin.xacro"/>
+  <xacro:include filename="$(find  lift_robot_description)/robots/lift_robot.urdf_origin.xacro"/>
   <xacro:include filename="$(find yumi_description)/urdf/camera_base/camera_base.urdf.xacro"/>
+  <xacro:include filename="$(find realsense2_description)/urdf/_d435.urdf.xacro" />
   <xacro:property name="yumi_setup" value="$(arg yumi_setup)" />
   <xacro:if value="${yumi_setup == 'robot_centric'}">
@@ -40,3 +41,6 @@
   <origin xyz="-0.025 0.0 0.475 " rpy="0  0 0" />
 </xacro:camera_base>
+<xacro:sensor_d435 parent="camera_base_2_link" >
+  <origin xyz="0.1 0 -0.02" rpy="0 ${PI/2} 0"/>
+</xacro:sensor_d435>
 </robot>
