Commit message: [fix]can launch gazebo

File: yumi_description/urdf/yumi.urdf.xacro (robot description, xacro)
@@ -11,16 +11,4 @@
   <!-- Import Gazebo plugins -->
   <xacro:include filename="$(find yumi_description)/urdf/Gazebo/gazebo.urdf.xacro"/>
-  <!--yumi-->
-  <xacro:yumi name="yumi" hardware_interface="hardware_interface/$(arg arms_interface)" parent="${yumi_parent}" >
-    <origin xyz="0 0 0.1" rpy="0 0 0" />
-  </xacro:yumi>
-  <!--right gripper-->
-  <xacro:yumi_servo_gripper name="gripper_r" hardware_interface="hardware_interface/$(arg grippers_interface)" parent="yumi_link_7_r">
-    <origin xyz="0 0 0.007" rpy="0 0 ${PI}" />
-  </xacro:yumi_servo_gripper>
-  <!--left gripper-->
-  <xacro:yumi_servo_gripper name="gripper_l" hardware_interface="hardware_interface/$(arg grippers_interface)" parent="yumi_link_7_l">
-    <origin xyz="0 0 0.007" rpy="0 0 ${PI}" />
-  </xacro:yumi_servo_gripper>
   <xacro:property name="yumi_setup" value="$(arg yumi_setup)" />
   <xacro:if value="${yumi_setup == 'robot_centric'}">
@@ -36,3 +24,15 @@
     </joint>
   </xacro:if>
+  <!--yumi-->
+  <xacro:yumi name="yumi" hardware_interface="hardware_interface/$(arg arms_interface)" parent="${yumi_parent}" >
+    <origin xyz="0 0 0.1" rpy="0 0 0" />
+  </xacro:yumi>
+  <!--right gripper-->
+  <xacro:yumi_servo_gripper name="gripper_r" hardware_interface="hardware_interface/$(arg grippers_interface)" parent="yumi_link_7_r">
+    <origin xyz="0 0 0.007" rpy="0 0 ${PI}" />
+  </xacro:yumi_servo_gripper>
+  <!--left gripper-->
+  <xacro:yumi_servo_gripper name="gripper_l" hardware_interface="hardware_interface/$(arg grippers_interface)" parent="yumi_link_7_l">
+    <origin xyz="0 0 0.007" rpy="0 0 ${PI}" />
+  </xacro:yumi_servo_gripper>
 </robot>

Commit message: [add]lift_robot model union

File: yumi_description/urdf/yumi.urdf.xacro (robot description, xacro)
@@ -11,4 +11,5 @@
   <!-- Import Gazebo plugins -->
   <xacro:include filename="$(find yumi_description)/urdf/Gazebo/gazebo.urdf.xacro"/>
+    <xacro:include filename="$(find  lift_robot_description)/robots/lift_robot.urdf_origin.xacro"/>
   <xacro:property name="yumi_setup" value="$(arg yumi_setup)" />
   <xacro:if value="${yumi_setup == 'robot_centric'}">
@@ -16,10 +17,9 @@
   </xacro:if>
   <xacro:if value="${yumi_setup == 'default'}">
-    <xacro:property name="yumi_parent" value="world" />
-    <link name="world"/>
-    <joint name="world_joint" type="fixed">
-      <parent link="world"/>
+    <xacro:property name="yumi_parent" value="base_link_to_world_joint" />
+    <joint name="base_link_to_world_joint" type="fixed">
+      <parent link="connect_base_link"/>
       <child link="yumi_base_link"/>
-      <origin xyz="0 0 0.1" rpy="0 0 0" />
+      <origin xyz="0 0 0.015" />
     </joint>
   </xacro:if>

Commit message: [add]camera_base in simulation

File: yumi_description/urdf/yumi.urdf.xacro (robot description, xacro)
@@ -12,4 +12,5 @@
   <xacro:include filename="$(find yumi_description)/urdf/Gazebo/gazebo.urdf.xacro"/>
     <xacro:include filename="$(find  lift_robot_description)/robots/lift_robot.urdf_origin.xacro"/>
+  <xacro:include filename="$(find yumi_description)/urdf/camera_base/camera_base.urdf.xacro"/>
   <xacro:property name="yumi_setup" value="$(arg yumi_setup)" />
   <xacro:if value="${yumi_setup == 'robot_centric'}">
@@ -36,3 +37,6 @@
     <origin xyz="0 0 0.007" rpy="0 0 ${PI}" />
   </xacro:yumi_servo_gripper>
+<xacro:camera_base parent="yumi_base_link" angle="${- PI/4}">
+  <origin xyz="-0.025 0.0 0.475 " rpy="0  0 0" />
+</xacro:camera_base>
 </robot>

Commit message: [modify]adjust lift_robot's prop position and yumi

File: yumi_description/urdf/yumi.urdf.xacro (robot description, xacro)
@@ -23,5 +23,5 @@
       <parent link="connect_base_link"/>
       <child link="yumi_base_link"/>
-      <origin xyz="0 0 0.015" />
+      <origin xyz="0.255 0 0.106" />
     </joint>
   </xacro:if>

Commit message: [Adjust]camera angle to 60 degrees.

File: yumi_description/urdf/yumi.urdf.xacro (robot description, xacro)
@@ -38,9 +38,9 @@
     <origin xyz="0 0 0.007" rpy="0 0 ${PI}" />
   </xacro:yumi_servo_gripper>
-<xacro:camera_base parent="yumi_base_link" angle="${- PI/4}">
+<xacro:camera_base parent="yumi_base_link" angle="${-PI/3}">
   <origin xyz="-0.025 0.0 0.475 " rpy="0  0 0" />
 </xacro:camera_base>
 <xacro:sensor_zed parent="camera_base_2_link" >
-  <origin xyz="0.1 0 -0.02" rpy="0 ${PI/2} 0"/>
+  <origin xyz="0.15 0 -0.03" rpy="0 ${PI/2} 0"/>
 </xacro:sensor_zed>
 </robot>
