Commit message: [Add]using Moveit in real space

File: yumi_description/urdf/yumi.urdf (robot description, URDF)
Before this commit: robot yumi, 22 links, 21 joints
Links:
- added link base_footprint
- added link camera_base_2_link, mass 0.25; collision box size=0.25 0.015 0.015; visual mesh filename=package://yumi_description/meshes/camera_base/yumi_camera_b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
- added link camera_base_link, mass 0.2; collision box size=0.15 0.015 0.015; visual mesh filename=package://yumi_description/meshes/camera_base/yumi_camera_b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
- added link connect_base_link, mass 0.434; collision box size=0.17 0.17 0.015; visual mesh filename=package://lift_robot_description/meshes/stl/connect_base_v2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
- added link front_left_steering_link, mass 2.29; collision cylinder length=0.0816 radius=0.0725; visual mesh filename=package://lift_robot_description/meshes/stl/4s2w_steering_v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
- added link front_left_wheel_link, mass 5.0; collision cylinder length=0.016 radius=0.025; visual mesh filename=package://lift_robot_description/meshes/stl/4s2w_wheel_v1.S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
- added link front_right_steering_link, mass 2.29; collision cylinder length=0.0816 radius=0.0725; visual mesh filename=package://lift_robot_description/meshes/stl/4s2w_steering_v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
- added link front_right_wheel_link, mass 5.0; collision cylinder length=0.016 radius=0.025; visual mesh filename=package://lift_robot_description/meshes/stl/4s2w_wheel_v1.S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
- added link hokuyo_link; collision box size=0.05 0.05 0.05; visual box size=0.05 0.05 0.05
- added link prop_link, mass 2.813; collision box size=0.075 0.075 0.5; visual box size=0.075 0.075 0.5
- added link rear_left_steering_link, mass 2.29; collision cylinder length=0.0816 radius=0.0725; visual mesh filename=package://lift_robot_description/meshes/stl/4s2w_steering_v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
- added link rear_left_wheel_link, mass 5.0; collision cylinder length=0.016 radius=0.025; visual mesh filename=package://lift_robot_description/meshes/stl/4s2w_wheel_v1.S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
- added link rear_right_steering_link, mass 2.29; collision cylinder length=0.0816 radius=0.0725; visual mesh filename=package://lift_robot_description/meshes/stl/4s2w_steering_v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
- added link rear_right_wheel_link, mass 5.0; collision cylinder length=0.016 radius=0.025; visual mesh filename=package://lift_robot_description/meshes/stl/4s2w_wheel_v1.S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
- added link under_base_link, mass 153.51; collision box size=0.45 0.45 0.116; visual mesh filename=package://lift_robot_description/meshes/stl/4s2w_under_base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
- added link zed_camera_center, mass 0.564; collision box size=0.02505 0.090 0.025; visual mesh filename=package://zed_wrapper/urdf/models/zed.stl
- added link zed_color_frame
- added link zed_color_optical_frame
- added link zed_depth_frame
- added link zed_depth_optical_frame
- added link zed_left_camera_frame
- added link zed_left_camera_optical_frame
- added link zed_right_camera_frame
- added link zed_right_camera_optical_frame
- link gripper_l_finger_l: mass 0.01 -> 0.04
- link gripper_l_finger_r: mass 0.01 -> 0.04
- link gripper_r_finger_l: mass 0.01 -> 0.04
- link gripper_r_finger_r: mass 0.01 -> 0.04
Joints:
- added joint base_link_to_world_joint: type fixed, parent connect_base_link, child yumi_base_link, origin xyz=0.255 0 0.106
- added joint camera_base_link_joint: type fixed, parent yumi_base_link, child camera_base_link, origin xyz=-0.025 0.0 0.475  rpy=0  0 0
- added joint camera_base_link_joint_2: type fixed, parent camera_base_link, child camera_base_2_link, origin xyz=0.075 0.0 0 rpy=0.0 -1.0471975512 0.0
- added joint connect_base_link_joint: type prismatic, parent prop_link, child connect_base_link, origin xyz=0.1455 0 0.025 rpy=0 0 0, axis 0 0 1, limit lower=0 upper=0.465 effort=1000.0 velocity=0.5
- added joint front_left_steering_joint: type revolute, parent under_base_link, child front_left_steering_link, origin xyz=0.14 0.14  0.012 rpy=0.0 0.0 3.14159274, axis 0 0 1, limit lower=-314.159274 upper=314.159274 effort=10000 velocity=0.05
- added joint front_left_wheel_joint: type continuous, parent front_left_steering_link, child front_left_wheel_link, origin xyz=0 -0.025 0 rpy=0.0 0.0 0.0, axis 0 -1 0, limit effort=200 velocity=10.0
- added joint front_right_steering_joint: type revolute, parent under_base_link, child front_right_steering_link, origin xyz=0.14 -0.14   0.012 rpy=0 0 0, axis 0 0 1, limit lower=-314.159274 upper=314.159274 effort=10000 velocity=0.05
- added joint front_right_wheel_joint: type continuous, parent front_right_steering_link, child front_right_wheel_link, origin xyz=0 -0.025 0 rpy=0.0 0.0 0.0, axis 0 1 0, limit effort=200 velocity=10.0
- added joint hokuyo_joint: type fixed, parent under_base_link, child hokuyo_link, origin xyz=0.2 0 0.0775 rpy=0 0 0
- added joint prop_to_base_link_joint: type fixed, parent under_base_link, child prop_link, origin xyz=-0.1775 0 0.1 rpy=0 0 0
- added joint rear_left_steering_joint: type revolute, parent under_base_link, child rear_left_steering_link, origin xyz=-0.14 0.14  0.012  rpy=0.0 0.0 3.14159274, axis 0 0 1, limit lower=-314.159274 upper=314.159274 effort=10000 velocity=0.05
- added joint rear_left_wheel_joint: type continuous, parent rear_left_steering_link, child rear_left_wheel_link, origin xyz=0 -0.025 0 rpy=0.0 0.0 0.0, axis 0 -1 0, limit effort=200 velocity=10.0
- added joint rear_right_steering_joint: type revolute, parent under_base_link, child rear_right_steering_link, origin xyz=-0.14 -0.14  0.012 rpy=0 0 0, axis 0 0 1, limit lower=-314.159274 upper=314.159274 effort=10000 velocity=0.05
- added joint rear_right_wheel_joint: type continuous, parent rear_right_steering_link, child rear_right_wheel_link, origin xyz=0 -0.025 0 rpy=0.0 0.0 0.0, axis 0 1 0, limit effort=200 velocity=10.0
- added joint under_base_link_joint: type fixed, parent base_footprint, child under_base_link, origin xyz=0 0 0.013
- added joint zed_camera_center_joint: type fixed, parent camera_base_2_link, child zed_camera_center, origin xyz=0.15 0 -0.03 rpy=0 1.57079632679 0
- added joint zed_color_joint: type fixed, parent zed_camera_center, child zed_color_frame, origin xyz=0 0 0 rpy=0 0 0
- added joint zed_color_optical_joint: type fixed, parent zed_color_frame, child zed_color_optical_frame, origin xyz=0 0 0 rpy=-1.57079632679 0.0 -1.57079632679
- added joint zed_depth_joint: type fixed, parent zed_camera_center, child zed_depth_frame, origin xyz=0 0 0 rpy=0 0 0
- added joint zed_depth_optical_joint: type fixed, parent zed_depth_frame, child zed_depth_optical_frame, origin xyz=0 0 0 rpy=-1.57079632679 0.0 -1.57079632679
- added joint zed_left_camera_joint: type fixed, parent zed_camera_center, child zed_left_camera_frame, origin xyz=0 0.06 0 rpy=0 0 0
- added joint zed_left_camera_optical_joint: type fixed, parent zed_left_camera_frame, child zed_left_camera_optical_frame, origin xyz=0 0 0 rpy=-1.57079632679 0.0 -1.57079632679
- added joint zed_right_camera_joint: type fixed, parent zed_camera_center, child zed_right_camera_frame, origin xyz=0 -0.06 0 rpy=0 0 0
- added joint zed_right_camera_optical_joint: type fixed, parent zed_right_camera_frame, child zed_right_camera_optical_frame, origin xyz=0 0 0 rpy=-1.57079632679 0.0 -1.57079632679
